Commit message: First commit with working hardware interface

File: robot-arm/ws_moveit/src/brc_arm/brc_arm_description/urdf/brc_arm_description.urdf (robot description, URDF)
Before this commit: robot brc_arm_description, 8 links, 7 joints
Links:
- added link LFinger, mass 0.052748844949343; collision mesh filename=package://brc_arm_description/meshes/LFinger.STL; visual mesh filename=package://brc_arm_description/meshes/LFinger.STL
- added link LLink1, mass 0.00668722339297275; collision mesh filename=package://brc_arm_description/meshes/LLink1.STL; visual mesh filename=package://brc_arm_description/meshes/LLink1.STL
- added link RFinger, mass 0.052748844949343; collision mesh filename=package://brc_arm_description/meshes/RFinger.STL; visual mesh filename=package://brc_arm_description/meshes/RFinger.STL
- added link RLink1, mass 0.00668722339297274; collision mesh filename=package://brc_arm_description/meshes/RLink1.STL; visual mesh filename=package://brc_arm_description/meshes/RLink1.STL
- link EEbase: mass 0.09260447609595 -> 0.0926044760959501
- link midarm1: mass 0.989206914918607 -> 0.836203235137727
- link midarm2: mass 0.141963495408494 -> 0.0646775902886999
- link wrist1: mass 0.488568583470577 -> 0.419666572951628
- link wrist2: mass 0.195554532888646 -> 0.129512939632169
Joints:
- added joint LFingerJ: type revolute, parent LLink1, child LFinger, origin xyz=-0.079999999999994 0 0 rpy=-1.5707963267949 0 0, axis 0 0 1, limit lower=0 upper=0 effort=0 velocity=0, mimic joint=LLink1J multiplier=-1 offset=0
- added joint LLink1J: type revolute, parent EEbase, child LLink1, origin xyz=-0.024 -0.011 -0.019185 rpy=0 0 0, axis 0 1 0, limit lower=0 upper=0 effort=0 velocity=0, mimic joint=RLink1J multiplier=1 offset=0
- added joint RFingerJ: type revolute, parent RLink1, child RFinger, origin xyz=0.0800000000000002 0 0 rpy=-1.5707963267949 0 3.14159265358979, axis 0 0 1, limit lower=0 upper=0 effort=0 velocity=0, mimic joint=RLink1J multiplier=-1 offset=0
- added joint RLink1J: type revolute, parent EEbase, child RLink1, origin xyz=0.024 -0.011 -0.019185 rpy=0 0 0, axis 0 1 0, limit lower=0 upper=6.283 effort=0 velocity=0
- joint EEbaseJ: limit lower=0 upper=0 effort=100 velocity=5 -> lower=0 upper=0 effort=0 velocity=0
- joint carriageJ: limit lower=0 upper=0.885 effort=150 velocity=5 -> lower=0 upper=0.885 effort=0 velocity=0
- joint midarm1J: limit lower=0 upper=6.283 effort=100 velocity=5 -> lower=0 upper=6.283 effort=0 velocity=0
- joint midarm2J: limit lower=0 upper=6.283 effort=100 velocity=5 -> lower=0 upper=6.283 effort=0 velocity=0
- joint wrist1J: limit lower=0 upper=1.57079632679 effort=100 velocity=5 -> lower=0 upper=6.283 effort=0 velocity=0; type revolute -> continuous
- joint wrist2J: limit lower=0 upper=6.283 effort=100 velocity=5 -> lower=0 upper=6.283 effort=0 velocity=0

Commit message: added teleop servoing

File: robot-arm/ws_moveit/src/brc_arm/brc_arm_description/urdf/brc_arm_description.urdf (robot description, URDF)
Before this commit: robot brc_arm_description, 12 links, 11 joints
Joints:
- joint LLink1J: mimic joint=RLink1J multiplier=1 offset=0 -> joint=RLink1J multiplier=-1 offset=0

Commit message: Added usb joystick support

File: robot-arm/ws_moveit/src/brc_arm/brc_arm_description/urdf/brc_arm_description.urdf (robot description, URDF)
Before this commit: robot brc_arm_description, 12 links, 11 joints
Links:
- link EEbase: mass 0.0926044760959501 -> 0.0926044760959502
- link LLink1: mass 0.00668722339297275 -> 0.00668722339297277
- link RLink1: mass 0.00668722339297274 -> 0.00668722339297277
- link base_link: mass 5.45066325397829 -> 127.989800714743
- link midarm1: mass 0.836203235137727 -> 0.836203235137726
- link midarm2: mass 0.0646775902886999 -> 0.0646775902886998
Joints:
- joint EEbaseJ: limit lower=0 upper=0 effort=0 velocity=0 -> lower=0 upper=0 effort=0 velocity=10
- joint LFingerJ: limit lower=0 upper=0 effort=0 velocity=0 -> lower=0 upper=0 effort=0 velocity=10; origin xyz=-0.079999999999994 0 0 rpy=-1.5707963267949 0 0 -> xyz=-0.08 0 0 rpy=-1.5708 0 0
- joint LLink1J: limit lower=0 upper=0 effort=0 velocity=0 -> lower=0 upper=0 effort=0 velocity=10; origin xyz=-0.024 -0.011 -0.019185 rpy=0 0 0 -> xyz=-0.024 -0.011 -0.014095 rpy=0 0 0
- joint RFingerJ: limit lower=0 upper=0 effort=0 velocity=0 -> lower=0 upper=0 effort=0 velocity=10; origin xyz=0.0800000000000002 0 0 rpy=-1.5707963267949 0 3.14159265358979 -> xyz=0.08 0 0 rpy=-1.5708 0 -3.1416
- joint RLink1J: limit lower=0 upper=6.283 effort=0 velocity=0 -> lower=0 upper=6.283 effort=0 velocity=10; origin xyz=0.024 -0.011 -0.019185 rpy=0 0 0 -> xyz=0.024 -0.011 -0.014095 rpy=0 0 0
- joint carriageJ: limit lower=0 upper=0.885 effort=0 velocity=0 -> lower=0 upper=0.885 effort=0 velocity=10
- joint midarm1J: limit lower=0 upper=6.283 effort=0 velocity=0 -> lower=0 upper=2.7423 effort=0 velocity=10; origin xyz=0 0 0.1 rpy=0 1.5708 0 -> xyz=0 0 0.1 rpy=0 0.5236 0; type continuous -> revolute
- joint midarm2J: axis 0 1 0 -> 0 -1 0; limit lower=0 upper=6.283 effort=0 velocity=0 -> lower=0 upper=4.8945 effort=0 velocity=10; origin xyz=-0.35 0 0 rpy=0 0 -3.1416 -> xyz=-0.35 0 0 rpy=0 -0.43633 0; type continuous -> revolute
- joint wrist1J: axis 0 0 1 -> 0 0 -1; limit lower=0 upper=6.283 effort=0 velocity=0 -> lower=0 upper=1.57 effort=0 velocity=10; origin xyz=0.08 -0.025 0 rpy=0 0 0 -> xyz=0.08 0.025 0 rpy=0 0 0; type continuous -> revolute
- joint wrist2J: limit lower=0 upper=6.283 effort=0 velocity=0 -> lower=0 upper=4.165 effort=0 velocity=10; origin xyz=0.225 0 0 rpy=-3.1416 0 0 -> xyz=0.225 0 0 rpy=-3.1416 -1.2217 3.1416; type continuous -> revolute

Commit message: Fix end effector finger joints

File: robot-arm/ws_moveit/src/brc_arm/brc_arm_description/urdf/brc_arm_description.urdf (robot description, URDF)
Before this commit: robot brc_arm_description, 12 links, 11 joints
Joints:
- joint LFingerJ: mimic joint=LLink1J multiplier=-1 offset=0 -> joint=RLink1J multiplier=1 offset=0
- joint RFingerJ: mimic joint=RLink1J multiplier=-1 offset=0 -> joint=RLink1J multiplier=1 offset=0

Commit message: Add support for end effector

File: robot-arm/ws_moveit/src/brc_arm/brc_arm_description/urdf/brc_arm_description.urdf (robot description, URDF)
Before this commit: robot brc_arm_description, 12 links, 11 joints
Joints:
- joint RLink1J: limit lower=0 upper=6.283 effort=0 velocity=10 -> lower=0 upper=1.22 effort=0 velocity=10

Commit message: updated urdf joint origins and limits

File: robot-arm/ws_moveit/src/brc_arm/brc_arm_description/urdf/brc_arm_description.urdf (robot description, URDF)
Before this commit: robot brc_arm_description, 12 links, 11 joints
Joints:
- joint midarm1J: origin xyz=0 0 0.1 rpy=0 0.5236 0 -> xyz=0 0 0.1 rpy=0 0.2932 0
- joint midarm2J: limit lower=0 upper=4.8945 effort=0 velocity=10 -> lower=0 upper=4.1887 effort=0 velocity=10; origin xyz=-0.35 0 0 rpy=0 -0.43633 0 -> xyz=-0.35 0 0 rpy=0 -0.9826 0
